File: minibee/revF_kicad/MiniBee.sch (KiCad schematic (older format))
At the start: 38 parts, among them IC1 MEGA8-AI, U1 ADXL345

Commit message: updates to board: exchanged D2 and D7, other switch
Parts:
- removed SWITCH12: MYSHIT_PCM_SWITCH, MiniBee:MINIBEE_MYSHIT_PCM_SWITCH_RA, symbol MINIBEE_MYSHIT_PCM_SWITCH
- added SW1: Switch_SPDT_x2, alps:alps_switch, symbol Switch_SPDT_x2
Connections:
- net labels added: D2
Other:
- note removed: "E"
- note removed: "Sense/Stage"
- note removed: "https://www.sensestage.eu"
- moved on the sheet: C1, C2, C3, C4, C5, F1, IC1, JP1, JP10, JP11, JP12, JP13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
